File: electrical/mazda-auxmod-pcb/mazda-auxmod-pcb.kicad_sch (KiCad schematic)
At the start: 33 parts, among them J1 Conn_01x15_Shielded, J2 Conn_01x10, J3 AudioJack4_Ground, J4 Conn_01x03, Q1 2N3904, Q2 2N3904, Q3 2SA715, U1 ATtiny45-20P, U2 L78L05_TO92, U3 L7805

Commit message: Added Schematic PDF
Parts:
- J3: footprint Connector_Audio:Jack_3.5mm_PJ320E_Horizontal -> Connector_Audio:Jack_3.5mm_PJ320D_Horizontal
Other:
- company: (none) -> Andrew Wilson
- title: (none) -> Mazda AuxMod
Changed lines of the file:
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@@
 (kicad_sch (version 20230121) (generator eeschema)
   (paper "A4")
+  (title_block
+    (title "Mazda AuxMod")
+    (date "2024-04-06")
+    (rev "v1.0")
+    (company "Andrew Wilson")
+    (comment 1 "www.github.com/andrewandneil/mazda-auxmod")
+  )
   (junction (at 59.69 176.53) (diameter 0) (color 0 0 0 0)
   )
@@
   (no_connect (at 163.83 113.03))
   (no_connect (at 41.91 163.83))
-  (no_connect (at 39.37 124.46))
+  (no_connect (at 41.91 124.46))
   (no_connect (at 57.15 39.37))
   (no_connect (at 57.15 52.07))
@@
   )
   (wire (pts (xy 167.64 67.31) (xy 180.34 67.31))
+    (stroke (width 0) (type default))
+  )
+  (wire (pts (xy 41.91 124.46) (xy 39.37 124.46))
     (stroke (width 0) (type default))
   )
@@
       (effects (font (size 1.27 1.27)))
     )
-    (property "Footprint" "Connector_Audio:Jack_3.5mm_PJ320E_Horizontal" (at 34.29 124.46 0)
-      (effects (font (size 1.27 1.27)) hide)
-    )
+    (property "Footprint" "Connector_Audio:Jack_3.5mm_PJ320D_Horizontal" (at 34.29 124.46 0)
+      (effects (font (size 1.27 1.27)) hide)
+    )
